File: projects/baro-bmp390/baro-bmp390.kicad_pcb (KiCad board)
At the start: 2 copper layers, 18 x 26 mm, 13 parts, among them J1 STEMMA-QT, U1 BMP390

Commit message: 9/6 update
Routing:
- net GND: track 2.09 -> 3.76 mm, vias 5 -> 10

Commit message: batch
Routing:
- net +3V3: vias 3 -> 2
Changed lines of the file:
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@@
 		(tags "capacitor")
 		(property "Reference" "C2"
-			(at 0 -1.16 0)
-			(layer "F.SilkS")
-			(effects
-				(font
-					(size 1 1)
-					(thickness 0.15)
+			(at 0 1.1 0)
+			(layer "F.SilkS")
+			(effects
+				(font
+					(size 0.8 0.8)
+					(thickness 0.12)
 				)
 			)
@@
 		(tags "capacitor")
 		(property "Reference" "C3"
-			(at 0 -1.43 0)
-			(layer "F.SilkS")
-			(effects
-				(font
-					(size 1 1)
-					(thickness 0.15)
+			(at 2.4 0 0)
+			(layer "F.SilkS")
+			(effects
+				(font
+					(size 0.8 0.8)
+					(thickness 0.12)
 				)
 			)
@@
 		(tags "fiducial")
 		(property "Reference" "FID1"
-			(at 0 -2.45 0)
-			(layer "F.SilkS")
-			(effects
-				(font
-					(size 1 1)
-					(thickness 0.15)
+			(at 0 2.2 0)
+			(layer "F.SilkS")
+			(effects
+				(font
+					(size 0.8 0.8)
+					(thickness 0.12)
 				)
 			)
@@
 		(tags "fiducial")
 		(property "Reference" "FID2"
-			(at 0 -2.45 0)
-			(layer "F.SilkS")
-			(effects
-				(font
-					(size 1 1)
-					(thickness 0.15)
+			(at 0 2.2 0)
+			(layer "F.SilkS")
+			(effects
+				(font
+					(size 0.8 0.8)
+					(thickness 0.12)
 				)
 			)
@@
 	)
 	(gr_text "rev1 Lee Taeho"
-		(at 19 198.5 0)
+		(at 19 195 0)
 		(layer "F.SilkS")
 		(effects
@@
 	)
 	(gr_text "BARO-BMP390"
-		(at 19 197 0)
+		(at 19 193.5 0)
 		(layer "F.SilkS")
 		(effects
 			(font
-				(size 1 1)
+				(size 0.8 0.8)
 				(thickness 0.15)
 			)
@@
 		(net "+3V3")
 	)
-	(via
-		(at 24.2 192.822)
-		(size 0.6)
-		(drill 0.3)
-		(layers "F.Cu" "B.Cu")
-		(net "+3V3")
-	)
