File: examples/usb-c-power/usb-c-power.kicad_pcb (KiCad board)
At the start: 2 copper layers, 60 x 40 mm, 10 parts, among them J1 USB4105-GF-A, J2 Fused 5 V OUT

Commit message: Resolve USB-C connector DRC with compatible manufacturer geometry
Parts:
- J1: value USB4105-GF-A -> USB4125-GF-A; footprint USBC:USB_C_Receptacle_GCT_USB4105-xx-A_16P_TopMnt_Horizontal -> USBC:USB_C_Receptacle_GCT_USB4125-xx-x_6P_TopMnt_Horizontal
- moved J1 0.27 mm to (63.0, 52.8)
Routing:
- net VBUS: track 17.9 -> 20.4 mm
- net GND: track 5.24 -> 7.36 mm
- net CC2: track 5.93 -> 7.32 mm
- net CC1: track 5.72 -> 6.91 mm
